File: Design ESP32/Design ESP32.kicad_pcb (KiCad board)
At the start: 2 copper layers, 6 parts, among them U1 ESP32-S3-WROOM-1, U2 AMS1117-3.3

Commit message: test
Parts:
- added C5: 1uF, Resistor_SMD:R_0805_2012Metric, F.Cu at (95.1, 87.5)
- added C6: 100nF, Capacitor_SMD:C_0805_2012Metric, F.Cu at (95.7, 79.5)
- added J1: USB_C_Receptacle_USB2.0_16P, Connector_USB:USB_C_Receptacle_GCT_USB4105-xx-A_16P_TopMnt_Horizontal, F.Cu at (136.8, 108.7)
- added J2: Conn_01x08_Pin, Connector_PinHeader_1.00mm:PinHeader_1x08_P1.00mm_Vertical, F.Cu at (153.5, 77.0)
- added R1: 10K, Capacitor_SMD:C_0805_2012Metric, F.Cu at (95.7, 82.5)
- added R2: 100R, Resistor_SMD:R_0805_2012Metric, F.Cu at (100.1, 79.5)
- added R3: 5.1K, Resistor_SMD:R_0805_2012Metric, F.Cu at (132.5, 116.1)
- added R4: 5.1K, Resistor_SMD:R_0805_2012Metric, F.Cu at (132.5, 119.1)
- added S1: TS-1088-AR02016, TS-1088-AR02016:SW_TS-1088-AR02016, F.Cu at (100.9, 83.5)
- added S2: TS-1088-AR02016, TS-1088-AR02016:SW_TS-1088-AR02016, F.Cu at (100.9, 88.0)
- moved C1 54.2 mm to (116.5, 77.5)
- moved U2 53.3 mm to (109.5, 98.5)
- moved C2 50.0 mm to (121.5, 77.5)
- moved C3 27.1 mm to (120.0, 101.5)
- moved C4 27.1 mm to (120.0, 104.5)
Connections:
- U1 pad 13: unconnected-(U1-USB_D--Pad13) -> D-
- U1 pad 14: unconnected-(U1-USB_D+-Pad14) -> D+
- U1 pad 28: unconnected-(U1-IO35-Pad28) -> Net-(J2-Pin_8)
- U1 pad 29: unconnected-(U1-IO36-Pad29) -> Net-(J2-Pin_7)
- U1 pad 3: unconnected-(U1-EN-Pad3) -> EN
- U1 pad 30: unconnected-(U1-IO37-Pad30) -> Net-(J2-Pin_6)
- U1 pad 31: unconnected-(U1-IO38-Pad31) -> Net-(J2-Pin_5)
- U1 pad 32: unconnected-(U1-IO39-Pad32) -> Net-(J2-Pin_4)
- U1 pad 33: unconnected-(U1-IO40-Pad33) -> Net-(J2-Pin_3)
- U1 pad 34: unconnected-(U1-IO41-Pad34) -> Net-(J2-Pin_2)
- U1 pad 35: unconnected-(U1-IO42-Pad35) -> Net-(J2-Pin_1)
Routing:
- net Net-(J2-Pin_8): track 0.00 -> 13.0 mm
- net Net-(J2-Pin_7): track 0.00 -> 12.8 mm
- net Net-(J2-Pin_6): track 0.00 -> 12.5 mm
- net Net-(J2-Pin_5): track 0.00 -> 12.1 mm
- net Net-(J2-Pin_4): track 0.00 -> 11.5 mm
- net Net-(J2-Pin_3): track 0.00 -> 11.3 mm
- net Net-(J2-Pin_2): track 0.00 -> 11.2 mm
- net Net-(J2-Pin_1): track 0.00 -> 10.9 mm
