File: hardware/Design ESP32/Design ESP32.kicad_pcb (KiCad board)
At the start: 2 copper layers, 53 x 30.8 mm, 16 parts, among them J1 USB_C_Receptacle_USB2.0_16P, J3 Conn_01x08_Pin, U1 ESP32-S3-WROOM-1, U2 AMS1117-3.3

Commit message: update footprint C1, C2
Parts:
- C1: footprint Capacitor_SMD:C_0805_2012Metric -> Capacitor_Tantalum_SMD:CP_EIA-2012-15_AVX-P
- C2: footprint Capacitor_SMD:C_0805_2012Metric -> Capacitor_Tantalum_SMD:CP_EIA-1608-10_AVX-L
Changed lines of the file:
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@@
 		)
 	)
-	(footprint "Capacitor_SMD:C_0805_2012Metric"
+	(footprint "Capacitor_Tantalum_SMD:CP_EIA-1608-10_AVX-L"
 		(layer "F.Cu")
 		(at 172.35 105.35 180)
-		(descr "Capacitor SMD 0805 (2012 Metric), square (rectangular) end terminal, IPC_7351 nominal, (Body size source: IPC-SM-782 page 76, https://www.pcb-3d.com/wordpress/wp-content/uploads/ipc-sm-782a_amendment_1_and_2.pdf, https://docs.google.com/spreadsheets/d/1BsfQQcO9C6DZCsRaXUlFlo91Tg2WpOkGARC1WS5S8t0/edit?usp=sharing), generated with kicad-footprint-generator")
-		(tags "capacitor")
+		(descr "Tantalum Capacitor SMD AVX-L (1608-10 Metric), IPC_7351 nominal, (Body size from: https://www.vishay.com/docs/48064/_t58_vmn_pt0471_1601.pdf), generated with kicad-footprint-generator")
+		(tags "capacitor tantalum")
 		(property "Reference" "C2"
-			(at 0 0 0)
+			(at 0 -1.48 180)
 			(layer "F.SilkS")
 			(effects
 				(font
-					(size 0.5 0.5)
-					(thickness 0.125)
+					(size 1 1)
+					(thickness 0.15)
 				)
 			)
 		)
 		(property "Value" "10uF"
-			(at 0 1.68 0)
+			(at 0 1.48 180)
 			(layer "F.Fab")
 			(effects
@@
 			)
 		)
-		(property "Footprint" "Capacitor_SMD:C_0805_2012Metric"
+		(property "Footprint" "Capacitor_Tantalum_SMD:CP_EIA-1608-10_AVX-L"
 			(at 0 0 180)
 			(unlocked yes)
@@
 		(attr smd)
 		(fp_line
-			(start -0.261252 0.735)
-			(end 0.261252 0.735)
+			(start 0.8 -0.785)
+			(end -1.51 -0.785)
 			(stroke
 				(width 0.12)
@@
 		)
 		(fp_line
-			(start -0.261252 -0.735)
-			(end 0.261252 -0.735)
+			(start -1.51 0.785)
+			(end 0.8 0.785)
 			(stroke
 				(width 0.12)
@@
 		)
 		(fp_line
-			(start 1.7 0.98)
-			(end -1.7 0.98)
+			(start -1.51 -0.785)
+			(end -1.51 0.785)
+			(stroke
+				(width 0.12)
+				(type solid)
+			)
+			(layer "F.SilkS")
+		)
+		(fp_line
+			(start 1.5 0.78)
+			(end -1.5 0.78)
 			(stroke
 				(width 0.05)
@@
 		)
 		(fp_line
-			(start 1.7 -0.98)
-			(end 1.7 0.98)
+			(start 1.5 -0.78)
+			(end 1.5 0.78)
 			(stroke
 				(width 0.05)
@@
 		)
 		(fp_line
-			(start -1.7 0.98)
-			(end -1.7 -0.98)
+			(start -1.5 0.78)
+			(end -1.5 -0.78)
 			(stroke
 				(width 0.05)
@@
 		)
 		(fp_line
-			(start -1.7 -0.98)
-			(end 1.7 -0.98)
+			(start -1.5 -0.78)
+			(end 1.5 -0.78)
 			(stroke
 				(width 0.05)
@@
 		)
 		(fp_line
-			(start 1 0.625)
-			(end -1 0.625)
+			(start 0.8 0.425)
+			(end 0.8 -0.425)
 			(stroke
 				(width 0.1)
@@
 		)
 		(fp_line
-			(start 1 -0.625)
-			(end 1 0.625)
+			(start 0.8 -0.425)
+			(end -0.5 -0.425)
 			(stroke
 				(width 0.1)
@@
 		)
 		(fp_line
-			(start -1 0.625)
-			(end -1 -0.625)
+			(start -0.5 -0.425)
+			(end -0.8 -0.125)
 			(stroke
 				(width 0.1)
@@
 		)
 		(fp_line
-			(start -1 -0.625)
-			(end 1 -0.625)
+			(start -0.8 0.425)
+			(end 0.8 0.425)
+			(stroke
+				(width 0.1)
+				(type solid)
+			)
+			(layer "F.Fab")
+		)
+		(fp_line
+			(start -0.8 -0.125)
+			(end -0.8 0.425)
 			(stroke
 				(width 0.1)
@@
 		)
 		(fp_text user "${REFERENCE}"
-			(at 0 0 0)
+			(at 0 0 180)
 			(layer "F.Fab")
 			(effects
 				(font
-					(size 0.5 0.5)
-					(thickness 0.08)
+					(size 0.4 0.4)
+					(thickness 0.06)
 				)
 			)
 		)
 		(pad "1" smd roundrect
-			(at -0.95 0 180)
-			(size 1 1.45)
+			(at -0.7125 0 180)
+			(size 1.075 1.05)
 			(layers "F.Cu" "F.Paste" "F.Mask")
-			(roundrect_rratio 0.25)
+			(roundrect_rratio 0.238095)
 			(net 37 "+5V")
 			(pintype "passive")
 		)
 		(pad "2" smd roundrect
-			(at 0.95 0 180)
-			(size 1 1.45)
+			(at 0.7125 0 180)
+			(size 1.075 1.05)
 			(layers "F.Cu" "F.Paste" "F.Mask")
-			(roundrect_rratio 0.25)
+			(roundrect_rratio 0.238095)
 			(net 36 "GND")
 			(pintype "passive")
 		)
-		(model "${KICAD8_3DMODEL_DIR}/Capacitor_SMD.3dshapes/C_0805_2012Metric.wrl"
+		(model "${KICAD8_3DMODEL_DIR}/Capacitor_Tantalum_SMD.3dshapes/CP_EIA-1608-10_AVX-L.wrl"
 			(offset
 				(xyz 0 0 0)
@@
 		)
 	)
-	(footprint "Capacitor_SMD:C_0805_2012Metric"
+	(footprint "Capacitor_Tantalum_SMD:CP_EIA-2012-15_AVX-P"
 		(layer "F.Cu")
 		(at 172.35 101.85 180)
-		(descr "Capacitor SMD 0805 (2012 Metric), square (rectangular) end terminal, IPC_7351 nominal, (Body size source: IPC-SM-782 page 76, https://www.pcb-3d.com/wordpress/wp-content/uploads/ipc-sm-782a_amendment_1_and_2.pdf, https://docs.google.com/spreadsheets/d/1BsfQQcO9C6DZCsRaXUlFlo91Tg2WpOkGARC1WS5S8t0/edit?usp=sharing), generated with kicad-footprint-generator")
-		(tags "capacitor")
+		(descr "Tantalum Capacitor SMD AVX-P (2012-15 Metric), IPC_7351 nominal, (Body size from: https://www.vishay.com/docs/40182/tmch.pdf), generated with kicad-footprint-generator")
+		(tags "capacitor tantalum")
 		(property "Reference" "C1"
-			(at 0 0 0)
+			(at 0 -1.58 180)
 			(layer "F.SilkS")
 			(effects
 				(font
-					(size 0.5 0.5)
-					(thickness 0.125)
+					(size 1 1)
+					(thickness 0.15)
 				)
 			)
 		)
 		(property "Value" "22uF"
-			(at 0 1.68 0)
+			(at 0 1.58 180)
 			(layer "F.Fab")
-			(hide yes)
 			(effects
 				(font
@@
 			)
 		)
-		(property "Footprint" "Capacitor_SMD:C_0805_2012Metric"
+		(property "Footprint" "Capacitor_Tantalum_SMD:CP_EIA-2012-15_AVX-P"
 			(at 0 0 180)
 			(unlocked yes)
@@
 		(attr smd)
 		(fp_line
-			(start -0.261252 0.735)
-			(end 0.261252 0.735)
+			(start 1 -0.785)
+			(end -1.71 -0.785)
 			(stroke
 				(width 0.12)
@@
 		)
 		(fp_line
-			(start -0.261252 -0.735)
-			(end 0.261252 -0.735)
+			(start -1.71 0.785)
+			(end 1 0.785)
 			(stroke
 				(width 0.12)
@@
 		)
 		(fp_line
-			(start 1.7 0.98)
-			(end -1.7 0.98)
+			(start -1.71 -0.785)
+			(end -1.71 0.785)
+			(stroke
+				(width 0.12)
+				(type solid)
+			)
+			(layer "F.SilkS")
+		)
+		(fp_line
+			(start 1.7 0.88)
+			(end -1.7 0.88)
 			(stroke
 				(width 0.05)
@@
 		)
 		(fp_line
-			(start 1.7 -0.98)
-			(end 1.7 0.98)
+			(start 1.7 -0.88)
+			(end 1.7 0.88)
 			(stroke
 				(width 0.05)
@@
 		)
 		(fp_line
-			(start -1.7 0.98)
-			(end -1.7 -0.98)
+			(start -1.7 0.88)
+			(end -1.7 -0.88)
 			(stroke
 				(width 0.05)
@@
 		)
 		(fp_line
-			(start -1.7 -0.98)
-			(end 1.7 -0.98)
+			(start -1.7 -0.88)
+			(end 1.7 -0.88)
 			(stroke
 				(width 0.05)
@@
 		(fp_line
 			(start 1 0.625)
-			(end -1 0.625)
+			(end 1 -0.625)
 			(stroke
 				(width 0.1)
@@
 		(fp_line
 			(start 1 -0.625)
-			(end 1 0.625)
+			(end -0.6875 -0.625)
+			(stroke
+				(width 0.1)
+				(type solid)
+			)
+			(layer "F.Fab")
+		)
+		(fp_line
+			(start -0.6875 -0.625)
+			(end -1 -0.3125)
 			(stroke
 				(width 0.1)
@@
 		(fp_line
 			(start -1 0.625)
-			(end -1 -0.625)
+			(end 1 0.625)
 			(stroke
 				(width 0.1)
@@
 		)
 		(fp_line
-			(start -1 -0.625)
-			(end 1 -0.625)
+			(start -1 -0.3125)
+			(end -1 0.625)
 			(stroke
 				(width 0.1)
@@
 		)
 		(fp_text user "${REFERENCE}"
-			(at 0 0 0)
+			(at 0 0 180)
 			(layer "F.Fab")
 			(effects
@@
 		)
 		(pad "1" smd roundrect
-			(at -0.95 0 180)
-			(size 1 1.45)
+			(at -0.8875 0 180)
+			(size 1.125 1.05)
 			(layers "F.Cu" "F.Paste" "F.Mask")
-			(roundrect_rratio 0.25)
+			(roundrect_rratio 0.238095)
 			(net 35 "+3V3")
 			(pintype "passive")
 		)
 		(pad "2" smd roundrect
-			(at 0.95 0 180)
-			(size 1 1.45)
+			(at 0.8875 0 180)
+			(size 1.125 1.05)
 			(layers "F.Cu" "F.Paste" "F.Mask")
-			(roundrect_rratio 0.25)
+			(roundrect_rratio 0.238095)
 			(net 36 "GND")
 			(pintype "passive")
 		)
-		(model "${KICAD8_3DMODEL_DIR}/Capacitor_SMD.3dshapes/C_0805_2012Metric.wrl"
+		(model "${KICAD8_3DMODEL_DIR}/Capacitor_Tantalum_SMD.3dshapes/CP_EIA-2012-15_AVX-P.wrl"
 			(offset
 				(xyz 0 0 0)
@@
 		(tags "resistor")
 		(property "Reference" "R2"
-			(at 0 0 360)
+			(at 0 0 0)
 			(layer "F.SilkS")
 			(effects
@@
 		)
 		(property "Value" "100R"
-			(at 0 1.65 360)
+			(at 0 1.65 0)
 			(layer "F.Fab")
 			(hide yes)
@@
 		)
 		(fp_text user "${REFERENCE}"
-			(at 0 0 360)
+			(at 0 0 0)
 			(layer "F.Fab")
 			(effects
@@
 		(polygon
 			(pts
-				(xy 160 84.4) (xy 213 84.4) (xy 213 115) (xy 160 115.2) (xy 160 84.4)
+				(xy 160 84.4) (xy 213 84.4) (xy 213 115) (xy 160 115.2)
 			)
 		)
